File: ergogen-reversible/output/pcbs/souffle_wireless.kicad_pcb (KiCad board)
At the start: 2 copper layers, 133.8 x 109.5 mm, 126 parts

Commit message: feat: redoing with two hands
Connections:
- MCU1 pad 10: R2 -> MCU1_10
- MCU1 pad 11: R3 -> MCU1_11
- MCU1 pad 12: R4 -> MCU1_12
- MCU1 pad 13: P10 -> MCU1_13
- MCU1 pad 14: P16 -> MCU1_14
- MCU1 pad 15: C5 -> MCU1_15
- MCU1 pad 16: C4 -> MCU1_16
- MCU1 pad 17: C3 -> MCU1_17
- MCU1 pad 18: C2 -> MCU1_18
- MCU1 pad 19: C1 -> MCU1_19
- MCU1 pad 20: C0 -> MCU1_20
- MCU1 pad 5: SDA -> MCU1_5
- MCU1 pad 6: SCL -> MCU1_6
- MCU1 pad 7: CS -> MCU1_7
- MCU1 pad 8: R0 -> MCU1_8
- MCU1 pad 9: R1 -> MCU1_9
Routing:
- net (no net): track 111.0 -> 333.1 mm
